File: FanBridge.sch (KiCad schematic (older format))
At the start: 11 parts, among them P1 CONN_01X01, P2 CONN_01X01, P3 CONN_01X04, Q1 IRF7309IPBF, Q2 2N7002, Q3 2N7002, Q4 IRF7309IPBF

Commit message: 17.08.2017
Parts:
- removed P3: CONN_01X04, symbol CONN_01X04
- added C1: C, ~, symbol C
- added P3, P4, P5, P6: CONN_1, symbol CONN_1
Connections:
- net +8V: now also C1.1
- net GND: now also C1.2
- net control-: now reaches Q1.2 (G), Q3.1 (G), R1.1
- net control-: now also P5.1
- net power+: now reaches Q1.5 (D2), Q1.6 (D1), Q1.7 (D2), Q1.8 (D1)
- net power+: now also P4.1
- net control+: now reaches Q2.1 (G), Q4.2 (G), R4.1
- net control+: now also P6.1
- net power-: now reaches Q4.5 (D2), Q4.6 (D1), Q4.7 (D2), Q4.8 (D1)
- net power-: now also P3.1
Changed lines of the file:
@@
 Sheet 1 1
 Title ""
-Date "15 aug 2017"
+Date "17 aug 2017"
 Rev ""
 Comp ""
@@
 $EndComp
 $Comp
-L +8V #PWR01
+L +8V #PWR3
 U 1 1 59859E1E
 P 2350 1150
-F 0 "#PWR01" H 2350 1000 50  0001 C CNN
+F 0 "#PWR3" H 2350 1000 50  0001 C CNN
 F 1 "+8V" H 2350 1290 50  0000 C CNN
 F 2 "" H 2350 1150 50  0000 C CNN
@@
 $EndComp
 $Comp
-L +8V #PWR02
+L +8V #PWR6
 U 1 1 59859E42
 P 2950 1050
-F 0 "#PWR02" H 2950 900 50  0001 C CNN
+F 0 "#PWR6" H 2950 900 50  0001 C CNN
 F 1 "+8V" H 2950 1190 50  0000 C CNN
 F 2 "" H 2950 1050 50  0000 C CNN
@@
 $EndComp
 $Comp
-L GND #PWR03
+L GND #PWR7
 U 1 1 59859E66
 P 2950 1650
-F 0 "#PWR03" H 2950 1400 50  0001 C CNN
+F 0 "#PWR7" H 2950 1400 50  0001 C CNN
 F 1 "GND" H 2950 1500 50  0000 C CNN
 F 2 "" H 2950 1650 50  0000 C CNN
@@
 $EndComp
 $Comp
-L GND #PWR04
+L GND #PWR4
 U 1 1 59859E8A
 P 2350 1950
-F 0 "#PWR04" H 2350 1700 50  0001 C CNN
+F 0 "#PWR4" H 2350 1700 50  0001 C CNN
 F 1 "GND" H 2350 1800 50  0000 C CNN
 F 2 "" H 2350 1950 50  0000 C CNN
@@
 $EndComp
 $Comp
-L +8V #PWR05
+L +8V #PWR11
 U 1 1 5985A773
 P 4450 1150
-F 0 "#PWR05" H 4450 1000 50  0001 C CNN
+F 0 "#PWR11" H 4450 1000 50  0001 C CNN
 F 1 "+8V" H 4450 1290 50  0000 C CNN
 F 2 "" H 4450 1150 50  0000 C CNN
@@
 $EndComp
 $Comp
-L +8V #PWR06
+L +8V #PWR8
 U 1 1 5985A779
 P 3850 1050
-F 0 "#PWR06" H 3850 900 50  0001 C CNN
+F 0 "#PWR8" H 3850 900 50  0001 C CNN
 F 1 "+8V" H 3850 1190 50  0000 C CNN
 F 2 "" H 3850 1050 50  0000 C CNN
@@
 $EndComp
 $Comp
-L GND #PWR07
+L GND #PWR9
 U 1 1 5985A77F
 P 3850 1650
-F 0 "#PWR07" H 3850 1400 50  0001 C CNN
+F 0 "#PWR9" H 3850 1400 50  0001 C CNN
 F 1 "GND" H 3850 1500 50  0000 C CNN
 F 2 "" H 3850 1650 50  0000 C CNN
@@
 $EndComp
 $Comp
-L GND #PWR08
+L GND #PWR12
 U 1 1 5985A785
 P 4450 1950
-F 0 "#PWR08" H 4450 1700 50  0001 C CNN
+F 0 "#PWR12" H 4450 1700 50  0001 C CNN
 F 1 "GND" H 4450 1800 50  0000 C CNN
 F 2 "" H 4450 1950 50  0000 C CNN
@@
 Wire Wire Line
 	3850 1250 4150 1250
-$Comp
-L CONN_01X04 P3
-U 1 1 5985A990
-P 3400 2650
-F 0 "P3" H 3400 2900 50  0000 C CNN
-F 1 "CONN_01X04" V 3500 2650 50  0000 C CNN
-F 2 "" H 3400 2650 50  0000 C CNN
-F 3 "" H 3400 2650 50  0000 C CNN
-	1    3400 2650
-	0    1    1    0
-$EndComp
 $Comp
 L CONN_01X01 P1
@@
 U 1 1 5985AB0A
 P 950 1750
-F 0 "P2" H 950 1850 50  0000 C CNN
+F 0 "P2" V 950 1850 50  0000 C CNN
 F 1 "CONN_01X01" V 1050 1750 50  0000 C CNN
 F 2 "" H 950 1750 50  0000 C CNN
@@
 $EndComp
 $Comp
-L +8V #PWR09
+L +8V #PWR1
 U 1 1 5985AB73
 P 750 1050
-F 0 "#PWR09" H 750 900 50  0001 C CNN
+F 0 "#PWR1" H 750 900 50  0001 C CNN
 F 1 "+8V" H 750 1190 50  0000 C CNN
 F 2 "" H 750 1050 50  0000 C CNN
@@
 $EndComp
 $Comp
-L GND #PWR010
+L GND #PWR2
 U 1 1 5985AB9D
 P 750 1750
-F 0 "#PWR010" H 750 1500 50  0001 C CNN
+F 0 "#PWR2" H 750 1500 50  0001 C CNN
 F 1 "GND" H 750 1600 50  0000 C CNN
 F 2 "" H 750 1750 50  0000 C CNN
@@
 $EndComp
 $Comp
-L GND #PWR011
+L GND #PWR10
 U 1 1 59871348
 P 4150 2000
-F 0 "#PWR011" H 4150 1750 50  0001 C CNN
+F 0 "#PWR10" H 4150 1750 50  0001 C CNN
 F 1 "GND" H 4150 1850 50  0000 C CNN
 F 2 "" H 4150 2000 50  0000 C CNN
@@
 $EndComp
 $Comp
-L GND #PWR012
+L GND #PWR5
 U 1 1 59871376
 P 2650 2200
-F 0 "#PWR012" H 2650 1950 50  0001 C CNN
+F 0 "#PWR5" H 2650 1950 50  0001 C CNN
 F 1 "GND" H 2650 2050 50  0000 C CNN
 F 2 "" H 2650 2200 50  0000 C CNN
@@
 Connection ~ 4550 1550
 Connection ~ 2250 1550
+$Comp
+L CONN_1 P3
+U 1 1 59955684
+P 3250 2600
+F 0 "P3" H 3330 2600 40  0000 L CNN
+F 1 "CONN_1" H 3250 2655 30  0001 C CNN
+F 2 "" H 3250 2600 60  0000 C CNN
+F 3 "" H 3250 2600 60  0000 C CNN
+	1    3250 2600
+	0    1    1    0
+$EndComp
+$Comp
+L CONN_1 P4
+U 1 1 59955693
+P 3350 2600
+F 0 "P4" H 3430 2600 40  0000 L CNN
+F 1 "CONN_1" H 3350 2655 30  0001 C CNN
+F 2 "" H 3350 2600 60  0000 C CNN
+F 3 "" H 3350 2600 60  0000 C CNN
+	1    3350 2600
+	0    1    1    0
+$EndComp
+$Comp
+L CONN_1 P5
+U 1 1 599556A2
+P 3450 2600
+F 0 "P5" H 3530 2600 40  0000 L CNN
+F 1 "CONN_1" H 3450 2655 30  0001 C CNN
+F 2 "" H 3450 2600 60  0000 C CNN
+F 3 "" H 3450 2600 60  0000 C CNN
+	1    3450 2600
+	0    1    1    0
+$EndComp
+$Comp
+L CONN_1 P6
+U 1 1 599556B1
+P 3550 2600
+F 0 "P6" H 3630 2600 40  0000 L CNN
+F 1 "CONN_1" H 3550 2655 30  0001 C CNN
+F 2 "" H 3550 2600 60  0000 C CNN
+F 3 "" H 3550 2600 60  0000 C CNN
+	1    3550 2600
+	0    1    1    0
+$EndComp
+Text Label 1750 2400 0    60   ~ 0
+power+
+Text Label 3450 2150 0    60   ~ 0
+control-
+Text Label 3600 1800 0    60   ~ 0
+control+
+Text Label 2900 2500 0    60   ~ 0
+power-
+$Comp
+L C C1
+U 1 1 59957431
+P 750 1250
+F 0 "C1" H 750 1350 40  0000 L CNN
+F 1 "C" H 756 1165 40  0000 L CNN
+F 2 "~" H 788 1100 30  0000 C CNN
+F 3 "~" H 750 1250 60  0000 C CNN
+	1    750  1250
+	1    0    0    -1
+$EndComp
+Wire Wire Line
+	750  1450 750  1750
 $EndSCHEMATC
