File: FanBridge.kicad_pcb (KiCad board)
At the start: 2 copper layers, 15.2 x 10.2 mm, 11 parts, among them P1 CONN_01X01, P2 CONN_01X01, P3 CONN_01X04, Q1 IRF7309IPBF, Q2 2N7002, Q3 2N7002, Q4 IRF7309IPBF

Commit message: 15.08.2017
Parts:
- Q2, Q4, R2, R4: moved to B.Cu
- moved Q4 27.9 mm to (101.6, 81.3), turned to 270 degrees
- moved P2 25.7 mm to (134.6, 71.1)
- moved Q1 22.9 mm to (125.7, 88.9), turned to 90 degrees
- moved R4 15.3 mm to (102.9, 77.5)
- moved P1 13.3 mm to (124.5, 71.1)
- moved Q2 9.25 mm to (108.0, 78.7), turned to 90 degrees
- moved R1 4.02 mm to (127.0, 92.7), turned to 180 degrees
- moved Q3 2.54 mm to (132.1, 91.4)
- moved R2 2.54 mm to (108.0, 82.5), turned to 180 degrees
- moved R3 1.80 mm to (132.1, 87.6)
Connections:
- P3 pad 3: Net-(P3-Pad3) -> N-000007
- P3 pad 4: Net-(P3-Pad4) -> N-000006
- Q1 pad 4: (no net) -> N-000004
- Q1 pad 5: Net-(P3-Pad3) -> N-000007
- Q1 pad 6: Net-(Q1-Pad6) -> N-000007
- Q1 pad 7: Net-(P3-Pad3) -> N-000007
- Q1 pad 8: Net-(Q1-Pad6) -> N-000007
- Q2 pad 3: Net-(Q2-Pad3) -> N-000004
- Q3 pad 3: Net-(Q3-Pad3) -> N-000008
- Q4 pad 4: (no net) -> N-000008
- Q4 pad 5: Net-(P3-Pad4) -> N-000006
- Q4 pad 6: Net-(Q4-Pad6) -> N-000006
- Q4 pad 7: Net-(P3-Pad4) -> N-000006
- Q4 pad 8: Net-(Q4-Pad6) -> N-000006
- R2 pad 2: Net-(Q2-Pad3) -> N-000004
- R3 pad 2: Net-(Q3-Pad3) -> N-000008
Routing:
- net N-000008: track 0.00 -> 8.36 mm
- net N-000001: track 0.00 -> 8.02 mm
- net GND: track 0.00 -> 6.83 mm
- net N-000007: track 0.00 -> 3.81 mm
- net +8V: track 0.00 -> 2.42 mm

Commit message: 17.08.2017
Parts:
- added C1: C, c_1206, F.Cu at (128.3, 71.1)
- added P4: CONN_1, PIN_ARRAY_1, F.Cu at (123.2, 67.3)
- added P5: CONN_1, PIN_ARRAY_1, F.Cu at (125.7, 72.0)
- added P6: CONN_1, PIN_ARRAY_1, F.Cu at (133.3, 72.4)
- P3: value CONN_01X04 -> CONN_1; footprint PIN_ARRAY_2X2 -> PIN_ARRAY_1
- moved P3 34.2 mm to (123.2, 64.8)
- moved R2 30.2 mm to (134.5, 68.2)
- moved Q4 29.9 mm to (128.0, 67.2)
- moved Q2 29.6 mm to (134.4, 65.3)
- moved R4 27.3 mm to (129.4, 71.1), turned to 0 degrees
- moved Q3 23.8 mm to (134.6, 67.8)
- moved Q1 23.0 mm to (128.3, 66.0)
- moved R3 23.0 mm to (134.6, 64.8)
- moved R1 21.9 mm to (130.8, 71.1), turned to 90 degrees
- moved P2 1.80 mm to (135.9, 72.4)
- moved P1 1.55 mm to (123.2, 72.0)
Connections:
- P3 pad 1: N-000005 (its old number) -> /power-
- Q1 pad 2: N-000001 -> /control-
- Q1 pad 5: N-000007 -> /power+
- Q1 pad 6: N-000007 -> /power+
- Q1 pad 7: N-000007 -> /power+
- Q1 pad 8: N-000007 -> /power+
- Q2 pad 1: N-000005 (its old number) -> /control+
- Q3 pad 1: N-000001 -> /control-
- Q4 pad 2: N-000005 (its old number) -> /control+
- Q4 pad 5: N-000006 -> /power-
- Q4 pad 6: N-000006 -> /power-
- Q4 pad 7: N-000006 -> /power-
- Q4 pad 8: N-000006 -> /power-
- R1 pad 1: N-000001 -> /control-
- R4 pad 1: N-000005 (its old number) -> /control+
Routing:
- net GND: track 6.83 -> 40.2 mm
- net +8V: track 2.42 -> 20.7 mm, vias 0 -> 1
- net /control+: track 0.00 -> 15.3 mm
- net /control-: track 0.00 -> 14.0 mm
- net N-000005: track 0.00 -> 12.4 mm, vias 0 -> 1
- net N-000001: track 8.02 -> 0.00 mm
- net /power+: track 0.00 -> 6.36 mm
- net /power-: track 0.00 -> 6.05 mm
- net N-000007: track 3.81 -> 0.00 mm
- net N-000004: track 8.36 -> 12.1 mm, vias 0 -> 1
- added copper zone on F.Cu, net +8V
- added copper zone on B.Cu, net GND
Other:
- net class Default: via_dia 0.889 -> 1
- net class Power added: clearance 0.254, trace_width 0.254, via_dia 1, via_drill 0.635

Commit message: 18.08.2017
Routing:
- net /power+: track 6.36 -> 7.63 mm
- net /power-: track 6.05 -> 6.58 mm
- added copper zone on F.Cu, net /power+
- added copper zone on B.Cu, net /power-
Other:
- net class Output added: clearance 0.254, trace_width 1, via_dia 1, via_drill 0.635
Changed lines of the file:
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@@
     (thickness 1.6)
     (drawings 4)
-    (tracks 89)
+    (tracks 90)
     (zones 0)
     (modules 15)
@@
     (last_trace_width 0.254)
     (trace_clearance 0.254)
-    (zone_clearance 0.508)
+    (zone_clearance 0.5)
     (zone_45_only no)
     (trace_min 0.254)
@@
     (pad_to_mask_clearance 0.2)
     (aux_axis_origin 0 0)
-    (visible_elements FFFE5FBF)
+    (visible_elements FFFE7FBF)
     (pcbplotparams
       (layerselection 3178497)
@@
     (uvia_drill 0.127)
     (add_net "")
-    (add_net +8V)
     (add_net /control+)
     (add_net /control-)
+    (add_net N-000004)
+    (add_net N-000005)
+  )
+  (net_class Output ""
+    (clearance 0.254)
+    (trace_width 1)
+    (via_dia 1)
+    (via_drill 0.635)
+    (uvia_dia 0.508)
+    (uvia_drill 0.127)
     (add_net /power+)
     (add_net /power-)
-    (add_net GND)
-    (add_net N-000004)
-    (add_net N-000005)
   )
   (net_class Power ""
@@
     (uvia_dia 0.508)
     (uvia_drill 0.127)
+    (add_net +8V)
+    (add_net GND)
   )
   (module c_1206 (layer F.Cu)
@@
   (gr_line (start 121.92 73.66) (end 121.92 63.5) (angle 90) (layer Edge.Cuts) (width 0.15))
   (gr_line (start 137.16 73.66) (end 121.92 73.66) (angle 90) (layer Edge.Cuts) (width 0.15))
-  (segment (start 128.27 67.818) (end 128.27 69.723) (width 0.254) (layer F.Cu) (net 1) (status 800000))
-  (segment (start 123.19 72.009) (end 123.19 71.501) (width 0.254) (layer F.Cu) (net 1) (status C00000))
-  (segment (start 123.19 71.501) (end 124.968 69.723) (width 0.254) (layer F.Cu) (net 1) (status 400000))
-  (segment (start 124.968 69.723) (end 128.27 69.723) (width 0.254) (layer F.Cu) (net 1) (status 800000))
+  (segment (start 128.27 67.818) (end 128.27 69.723) (width 0.254) (layer F.Cu) (net 1))
+  (segment (start 123.19 72.009) (end 123.19 71.501) (width 0.254) (layer F.Cu) (net 1))
+  (segment (start 123.19 71.501) (end 124.968 69.723) (width 0.254) (layer F.Cu) (net 1))
+  (segment (start 124.968 69.723) (end 128.27 69.723) (width 0.254) (layer F.Cu) (net 1))
   (segment (start 128.27 67.818) (end 130.81 67.818) (width 0.254) (layer B.Cu) (net 1))
   (via (at 128.27 67.818) (size 1) (layers F.Cu B.Cu) (net 1))
@@
   (segment (start 133.223 72.39) (end 130.81 71.12) (width 0.254) (layer B.Cu) (net 2) (status 10))
   (segment (start 133.30936 66.2305) (end 133.24586 66.294) (width 0.254) (layer B.Cu) (net 2) (status 30))
-  (segment (start 131.064 66.675) (end 130.175 66.675) (width 0.254) (layer F.Cu) (net 3) (status 400000))
-  (segment (start 129.413 68.326) (end 130.81 69.723) (width 0.254) (layer F.Cu) (net 3) (status 800000))
+  (segment (start 131.064 66.675) (end 130.175 66.675) (width 0.254) (layer F.Cu) (net 3))
+  (segment (start 129.413 68.326) (end 130.81 69.723) (width 0.254) (layer F.Cu) (net 3))
   (segment (start 129.413 67.437) (end 129.413 68.326) (width 0.254) (layer F.Cu) (net 3))
   (segment (start 130.175 66.675) (end 129.413 67.437) (width 0.254) (layer F.Cu) (net 3))
-  (segment (start 125.73 72.009) (end 126.619 71.12) (width 0.254) (layer F.Cu) (net 3) (status 400000))
+  (segment (start 125.73 72.009) (end 126.619 71.12) (width 0.254) (layer F.Cu) (net 3))
   (segment (start 126.619 71.12) (end 130.302 71.12) (width 0.254) (layer F.Cu) (net 3))
   (segment (start 130.302 71.12) (end 130.81 70.612) (width 0.254) (layer F.Cu) (net 3))
-  (segment (start 130.81 70.612) (end 130.81 69.723) (width 0.254) (layer F.Cu) (net 3) (status 800000))
+  (segment (start 130.81 70.612) (end 130.81 69.723) (width 0.254) (layer F.Cu) (net 3))
   (segment (start 133.56336 66.8655) (end 133.37286 66.675) (width 0.254) (layer F.Cu) (net 3) (status 30))
   (segment (start 133.37286 66.675) (end 131.064 66.675) (width 0.254) (layer F.Cu) (net 3) (status 10))
-  (segment (start 123.19 67.31) (end 124.841 67.31) (width 0.254) (layer F.Cu) (net 4) (status 400000))
-  (segment (start 124.841 67.31) (end 125.476 66.675) (width 0.254) (layer F.Cu) (net 4) (status 800000))
-  (segment (start 125.476 64.135) (end 125.476 65.405) (width 0.254) (layer F.Cu) (net 4) (status C00000))
-  (segment (start 125.476 65.405) (end 125.476 66.675) (width 0.254) (layer F.Cu) (net 4) (status C00000))
-  (segment (start 125.476 66.675) (end 125.476 67.945) (width 0.254) (layer F.Cu) (net 4) (status C00000))
-  (segment (start 123.19 64.77) (end 124.714 64.77) (width 0.254) (layer B.Cu) (net 5) (status 400000))
-  (segment (start 124.714 64.77) (end 125.222 65.278) (width 0.254) (layer B.Cu) (net 5) (status 800000))
-  (segment (start 125.222 65.278) (end 125.222 66.548) (width 0.254) (layer B.Cu) (net 5) (status C00000))
-  (segment (start 125.222 66.548) (end 125.222 67.818) (width 0.254) (layer B.Cu) (net 5) (status C00000))
-  (segment (start 125.222 67.818) (end 125.222 69.088) (width 0.254) (layer B.Cu) (net 5) (status C00000))
-  (segment (start 130.81 72.517) (end 128.27 72.517) (width 0.254) (layer F.Cu) (net 6) (status C00000))
+  (segment (start 123.19 67.31) (end 124.841 67.31) (width 1) (layer F.Cu) (net 4) (status 400000))
+  (segment (start 124.841 67.31) (end 125.476 66.675) (width 1) (layer F.Cu) (net 4) (status 800000))
+  (segment (start 125.476 66.675) (end 125.476 65.405) (width 1) (layer F.Cu) (net 4) (status C00000))
+  (segment (start 125.476 64.135) (end 125.476 65.405) (width 0.254) (layer F.Cu) (net 4))
+  (segment (start 125.476 65.405) (end 125.476 66.675) (width 0.254) (layer F.Cu) (net 4))
+  (segment (start 125.476 66.675) (end 125.476 67.945) (width 0.254) (layer F.Cu) (net 4))
+  (segment (start 125.222 67.818) (end 125.222 66.548) (width 1) (layer B.Cu) (net 5) (status C00000))
+  (segment (start 123.19 64.77) (end 123.444 64.77) (width 1) (layer B.Cu) (net 5) (status C00000))
+  (segment (start 123.444 64.77) (end 125.222 66.548) (width 1) (layer B.Cu) (net 5) (status C00000))
+  (segment (start 125.222 65.278) (end 125.222 66.548) (width 0.254) (layer B.Cu) (net 5))
+  (segment (start 125.222 67.818) (end 125.222 69.088) (width 0.254) (layer B.Cu) (net 5))
+  (segment (start 130.81 72.517) (end 128.27 72.517) (width 0.254) (layer F.Cu) (net 6))
   (segment (start 132.969 70.993) (end 132.334 70.993) (width 0.254) (layer F.Cu) (net 6))
   (segment (start 132.334 70.993) (end 131.318 72.517) (width 0.254) (layer F.Cu) (net 6) (status 20))
@@
   (segment (start 136.0805 64.3255) (end 136.398 64.643) (width 0.254) (layer B.Cu) (net 8))
   (zone (net 1) (net_name +8V) (layer F.Cu) (hatch full 0.508)
+    (connect_pads (clearance 0.75))
+    (min_thickness 0.254)
+    (fill (arc_segments 16) (thermal_gap 0.508) (thermal_bridge_width 0.508))
+    (polygon
+      (pts
+        (xy 125.984 63.881) (xy 125.984 69.85) (xy 121.92 69.85) (xy 121.92 73.66) (xy 137.16 73.66)
+        (xy 137.16 63.5) (xy 125.984 63.5)
+      )
+    )
+  )
+  (zone (net 6) (net_name GND) (layer B.Cu) (hatch edge 0.508)
+    (connect_pads (clearance 0.75))
+    (min_thickness 0.254)
+    (fill (arc_segments 16) (thermal_gap 0.508) (thermal_bridge_width 0.508))
+    (polygon
+      (pts
+        (xy 125.984 64.643) (xy 125.984 69.85) (xy 121.92 69.85) (xy 121.92 73.66) (xy 137.16 73.66)
+        (xy 137.16 63.5) (xy 125.984 63.5)
+      )
+    )
+  )
+  (zone (net 5) (net_name /power-) (layer B.Cu) (hatch edge 0.508)
+    (connect_pads (clearance 0.5))
+    (min_thickness 0.254)
+    (fill (arc_segments 16) (thermal_gap 0.508) (thermal_bridge_width 0.508))
+    (polygon
+      (pts
+        (xy 121.92 63.5) (xy 124.714 63.5) (xy 124.714 68.453) (xy 121.92 68.453)
+      )
+    )
+  )
+  (zone (net 4) (net_name /power+) (layer F.Cu) (hatch edge 0.508)
     (connect_pads (clearance 1))
     (min_thickness 0.254)
@@
     (polygon
       (pts
-        (xy 121.92 63.5) (xy 121.92 73.66) (xy 137.16 73.66) (xy 137.16 63.5)
+        (xy 121.92 63.5) (xy 124.714 63.5) (xy 124.714 68.453) (xy 121.92 68.453)
       )
     )
-  )
-  (zone (net 6) (net_name GND) (layer B.Cu) (hatch edge 0.508)
-    (connect_pads (clearance 1))
-    (min_thickness 0.254)
-    (fill (arc_segments 16) (thermal_gap 0.508) (thermal_bridge_width 0.508))
-    (polygon
-      (pts
-        (xy 121.92 63.5) (xy 121.92 73.66) (xy 137.16 73.66) (xy 137.16 63.5)
-      )
-    )

Commit message: 21.08.2017
Other:
- net class Default: via_drill 0.635 -> 0.2
- net class Output: via_drill 0.635 -> 0.2
- net class Power: via_drill 0.635 -> 0.2
- rule via_min_drill: 0.508 -> 0.2
Changed lines of the file:
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@@
     (24 Dwgs.User user)
     (25 Cmts.User user)
-    (26 Eco1.User user)
+    (26 Eco1.User user hide)
     (27 Eco2.User user)
     (28 Edge.Cuts user)
@@
     (edge_width 0.15)
     (via_size 1)
-    (via_drill 0.635)
+    (via_drill 0.2)
     (via_min_size 0.889)
-    (via_min_drill 0.508)
+    (via_min_drill 0.2)
     (uvia_size 0.508)
     (uvia_drill 0.127)
@@
     (mod_text_width 0.15)
     (pad_size 1.524 1.524)
-    (pad_drill 0.762)
+    (pad_drill 0.2)
     (pad_to_mask_clearance 0.2)
     (aux_axis_origin 0 0)
-    (visible_elements FFFE7FBF)
+    (visible_elements FFFE7FBB)
     (pcbplotparams
       (layerselection 3178497)
@@
     (trace_width 0.254)
     (via_dia 1)
-    (via_drill 0.635)
+    (via_drill 0.2)
     (uvia_dia 0.508)
     (uvia_drill 0.127)
@@
     (trace_width 1)
     (via_dia 1)
-    (via_drill 0.635)
+    (via_drill 0.2)
     (uvia_dia 0.508)
     (uvia_drill 0.127)
@@
     (trace_width 0.254)
     (via_dia 1)
-    (via_drill 0.635)
+    (via_drill 0.2)
     (uvia_dia 0.508)
     (uvia_drill 0.127)
@@
     (fp_line (start -1.27 1.27) (end -1.27 -1.27) (layer F.SilkS) (width 0.1524))
     (fp_line (start 1.27 -1.27) (end 1.27 1.27) (layer F.SilkS) (width 0.1524))
-    (pad 1 thru_hole rect (at 0 0) (size 1.524 1.524) (drill 1.016)
+    (pad 1 thru_hole rect (at 0 0) (size 1.524 1.524) (drill 0.2)
       (layers *.Cu *.Mask F.SilkS)
       (net 1 +8V)
@@
     (fp_line (start -1.27 1.27) (end -1.27 -1.27) (layer F.SilkS) (width 0.1524))
     (fp_line (start 1.27 -1.27) (end 1.27 1.27) (layer F.SilkS) (width 0.1524))
-    (pad 1 thru_hole rect (at 0 0) (size 1.524 1.524) (drill 1.016)
+    (pad 1 thru_hole rect (at 0 0) (size 1.524 1.524) (drill 0.2)
       (layers *.Cu *.Mask F.SilkS)
       (net 6 GND)
@@
     (fp_line (start -1.27 1.27) (end -1.27 -1.27) (layer F.SilkS) (width 0.1524))
     (fp_line (start 1.27 -1.27) (end 1.27 1.27) (layer F.SilkS) (width 0.1524))
-    (pad 1 thru_hole rect (at 0 0) (size 1.524 1.524) (drill 1.016)
+    (pad 1 thru_hole rect (at 0 0) (size 1.524 1.524) (drill 0.2)
       (layers *.Cu *.Mask F.SilkS)
       (net 4 /power+)
@@
     (fp_line (start -1.27 1.27) (end -1.27 -1.27) (layer F.SilkS) (width 0.1524))
     (fp_line (start 1.27 -1.27) (end 1.27 1.27) (layer F.SilkS) (width 0.1524))
-    (pad 1 thru_hole rect (at 0 0) (size 1.524 1.524) (drill 1.016)
+    (pad 1 thru_hole rect (at 0 0) (size 1.524 1.524) (drill 0.2)
       (layers *.Cu *.Mask F.SilkS)
       (net 3 /control-)
@@
     (fp_line (start -1.27 1.27) (end -1.27 -1.27) (layer F.SilkS) (width 0.1524))
     (fp_line (start 1.27 -1.27) (end 1.27 1.27) (layer F.SilkS) (width 0.1524))
-    (pad 1 thru_hole rect (at 0 0) (size 1.524 1.524) (drill 1.016)
+    (pad 1 thru_hole rect (at 0 0) (size 1.524 1.524) (drill 0.2)
       (layers *.Cu *.Mask F.SilkS)
       (net 2 /control+)
@@
     (fp_line (start -1.27 1.27) (end -1.27 -1.27) (layer F.SilkS) (width 0.1524))
     (fp_line (start 1.27 -1.27) (end 1.27 1.27) (layer F.SilkS) (width 0.1524))
-    (pad 1 thru_hole rect (at 0 0) (size 1.524 1.524) (drill 1.016)
+    (pad 1 thru_hole rect (at 0 0) (size 1.524 1.524) (drill 0.2)
       (layers *.Cu *.Mask F.SilkS)
       (net 5 /power-)
@@
   (segment (start 133.56336 66.8655) (end 133.37286 66.675) (width 0.254) (layer F.Cu) (net 3) (status 30))
   (segment (start 133.37286 66.675) (end 131.064 66.675) (width 0.254) (layer F.Cu) (net 3) (status 10))
-  (segment (start 123.19 67.31) (end 124.841 67.31) (width 1) (layer F.Cu) (net 4) (status 400000))
-  (segment (start 124.841 67.31) (end 125.476 66.675) (width 1) (layer F.Cu) (net 4) (status 800000))
-  (segment (start 125.476 66.675) (end 125.476 65.405) (width 1) (layer F.Cu) (net 4) (status C00000))
+  (segment (start 123.19 67.31) (end 124.841 67.31) (width 1) (layer F.Cu) (net 4))
+  (segment (start 124.841 67.31) (end 125.476 66.675) (width 1) (layer F.Cu) (net 4))
+  (segment (start 125.476 66.675) (end 125.476 65.405) (width 1) (layer F.Cu) (net 4))
   (segment (start 125.476 64.135) (end 125.476 65.405) (width 0.254) (layer F.Cu) (net 4))
   (segment (start 125.476 65.405) (end 125.476 66.675) (width 0.254) (layer F.Cu) (net 4))
   (segment (start 125.476 66.675) (end 125.476 67.945) (width 0.254) (layer F.Cu) (net 4))
-  (segment (start 125.222 67.818) (end 125.222 66.548) (width 1) (layer B.Cu) (net 5) (status C00000))
-  (segment (start 123.19 64.77) (end 123.444 64.77) (width 1) (layer B.Cu) (net 5) (status C00000))
-  (segment (start 123.444 64.77) (end 125.222 66.548) (width 1) (layer B.Cu) (net 5) (status C00000))
+  (segment (start 125.222 67.818) (end 125.222 66.548) (width 1) (layer B.Cu) (net 5))
+  (segment (start 123.19 64.77) (end 123.444 64.77) (width 1) (layer B.Cu) (net 5))
+  (segment (start 123.444 64.77) (end 125.222 66.548) (width 1) (layer B.Cu) (net 5))
   (segment (start 125.222 65.278) (end 125.222 66.548) (width 0.254) (layer B.Cu) (net 5))
   (segment (start 125.222 67.818) (end 125.222 69.088) (width 0.254) (layer B.Cu) (net 5))
